File: hardware/kicad/fusion/fusion.kicad_sch (KiCad schematic)
At the start: 0 parts

Commit message: KiCad project settings
Other:
- title: (none) -> Fusion
Changed lines of the file:
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@@
 (kicad_sch (version 20211123) (generator eeschema)
   (paper "A4")
+  (title_block
+    (title "Fusion")
+  )
   (sheet_instances
     (path "/" (page "1"))
